Commit message: feat: 更新elbow关节限位为±135°(±2.3562 rad)
🔧 主要修改:
• elbow关节限位从±90°(±1.5708 rad)扩展到±135°(±2.3562 rad)
• 与armv1_ws驱动的动态限位基础值保持一致
• 支持更大的工作范围，提高机械臂灵活性

📁 修改文件:
• models/recomoProto1-190/recomoProto1-190.urdf
  - joint4_elbow_pitch限位更新
  - 更新文档注释说明

💡 应用场景:
• URDF仿真环境(Gazebo、RViz等)
• 机器人可视化和建模

✅ 验证: 限位值与硬件驱动基础配置匹配

File: models/recomoProto1-190/recomoProto1-190.urdf (robot description, URDF)
Before this commit: robot recomoProto1-190, 14 links, 13 joints
Joints:
- joint joint4_elbow_pitch: limit lower=-1.5708 upper=1.5708 effort=30.0 velocity=0.5 -> lower=-2.3562 upper=2.3562 effort=30.0 velocity=0.5
- joint joint5_arm_pitch: limit lower=-1.5708 upper=1.5708 effort=30.0 velocity=0.5 -> lower=-2.3562 upper=2.3562 effort=30.0 velocity=0.5

Commit message: 修复joint1和joint3的axis方向
- joint1_gimbal_pitch: axis从[0 0 -1]改为[0 0 1]
- joint3_gimbal_yaw: axis从[0 0 -1]改为[0 0 1]
- 更新文档说明，添加修改记录（2026-02-05）

原因：这两个关节的实际运动方向与URDF标注方向相反，现已修正

File: models/recomoProto1-190/recomoProto1-190.urdf (robot description, URDF)
Before this commit: robot recomoProto1-190, 14 links, 13 joints
Joints:
- joint joint1_gimbal_pitch: axis 0 0 -1 -> 0 0 1
- joint joint3_gimbal_yaw: axis 0 0 -1 -> 0 0 1

Commit message: Update gimbal joint limits to match RS4 driver config
- Updated joint2_gimbal_roll: -235° to +90° (was -95° to +240°)
- Updated joint1_gimbal_pitch: -210° to +110° (was -112° to +214°)
- joint3_gimbal_yaw: remains -180° to +180° (unchanged)
- All limits now match hardware-validated DJI RS4 driver configuration
- Updated URDF header comments to document changes (2026-02-06)

File: models/recomoProto1-190/recomoProto1-190.urdf (robot description, URDF)
Before this commit: robot recomoProto1-190, 14 links, 13 joints
Joints:
- joint joint1_gimbal_pitch: limit lower=-1.9548 upper=3.7350 effort=10.0 velocity=0.5 -> lower=-3.6652 upper=1.9199 effort=10.0 velocity=0.5
- joint joint2_gimbal_roll: limit lower=-1.6581 upper=4.1888 effort=10.0 velocity=0.5 -> lower=-4.1015 upper=1.5708 effort=10.0 velocity=0.5
